Commit message: updated DDPGfD to be more accurate to the paper, added unit testing for DDPGfD.py, added logging functions to replay buffer and sim manager, added inertia to object model

File: demos/rl_demo/resources/object_models/2v2_mod/2v2_mod_cuboid_small.urdf (robot description, URDF)
Before this commit: robot 2v2_mod_cuboid_small, 1 links, 0 joints
Links:
- link 2v2_mod_cuboid_small: mass None -> 0.1
