Commit message: updated physics of object and plane to be more in line with real world

File: demos/rl_demo/resources/object_models/2v2_mod/2v2_mod_cuboid_small_old_properties.urdf (robot description, URDF)
Before this commit: robot 2v2_mod_cuboid_small, 1 links, 0 joints
Links:
- link 2v2_mod_cuboid_small: mass 0.3 -> 0.1
