Commit message: implemented hindsight experience replay, modified prioirty function, added functions to data analysis gui

File: demos/expert_demo/resources/2v2_nosensors/2v2_nosensors_limited.urdf (robot description, URDF)
Before this commit: robot 2v2_nosensors, 5 links, 4 joints
Joints:
- joint l_distal_pin: limit lower=-3.14 upper=3.14 effort=1000.0 velocity=0.5 -> lower=-3.14 upper=0 effort=1000.0 velocity=0.5
- joint l_prox_pin: limit lower=-3.14 upper=3.14 effort=1000.0 velocity=0.5 -> lower=-1.57 upper=1.57 effort=1000.0 velocity=0.5
- joint r_distal_pin: limit lower=-3.14 upper=3.14 effort=1000.0 velocity=0.5 -> lower=0 upper=3.14 effort=1000.0 velocity=0.5
- joint r_prox_pin: limit lower=-3.14 upper=3.14 effort=1000.0 velocity=0.5 -> lower=-1.57 upper=1.57 effort=1000.0 velocity=0.5

File: demos/expert_demo/resources/object_models/2v2_mod/2v2_mod_cylinder_small_alt.urdf (robot description, URDF)
Before this commit: robot 2v2_mod_cuboid_small, 1 links, 0 joints
Links:
- link 2v2_mod_cuboid_small: geometry collision mesh filename=obj_files/alt_small_cylinder2.obj scale=1 1 1; visual mesh filename=obj_files/alt_small_cylinder2.obj scale=1 1 1
