Commit message: added handA and updated RNN gui to work with it instead of old hand A. updated env and reset stuff to work with new hand

File: demos/rl_demo/resources/2v2_Hand_A/hand/2v2_50.50_50.50_1.1_53.urdf (robot description, URDF)
Before this commit: robot 2v2_65.35_65.35_1.1_53, 7 links, 6 joints
Joints:
- joint finger0_segment1_joint: origin xyz=0 0.0936 0 rpy=0 0 0 -> xyz=0 0.072 0 rpy=0 0 0
- joint finger1_segment1_joint: origin xyz=0 0.0936 0 rpy=0 0 0 -> xyz=0 0.072 0 rpy=0 0 0

File: demos/rl_demo/resources/NigelHands/2v2_50.50_50.50_1.1_53/hand/2v2_50.50_50.50_1.1_53.urdf (robot description, URDF)
Before this commit: robot 2v2_65.35_65.35_1.1_53, 7 links, 6 joints
Links:
- removed link finger0_sensor
- removed link finger1_sensor
- link finger0_segment0: mass 0.1 -> None
- link finger0_segment1: mass 0.1 -> None
- link finger1_segment0: mass 0.1 -> None
- link finger1_segment1: mass 0.1 -> None
- link palm: mass 1 -> None
Joints:
- removed joint finger0_sensor1_joint
- removed joint finger1_sensor2_joint
- joint finger0_segment1_joint: origin xyz=0 0.0936 0 rpy=0 0 0 -> xyz=0 0.072 0 rpy=0 0 0
- joint finger1_segment1_joint: origin xyz=0 0.0936 0 rpy=0 0 0 -> xyz=0 0.072 0 rpy=0 0 0

File: demos/rl_demo/resources/NigelHands/2v2_50.50_50.50_1.1_63/hand/2v2_50.50_50.50_1.1_63.urdf (robot description, URDF)
Before this commit: robot 2v2_65.35_65.35_1.1_53, 7 links, 6 joints
Links:
- removed link finger0_sensor
- removed link finger1_sensor
- link finger0_segment0: mass 0.1 -> None
- link finger0_segment1: mass 0.1 -> None
- link finger1_segment0: mass 0.1 -> None
- link finger1_segment1: mass 0.1 -> None
- link palm: mass 1 -> None
Joints:
- removed joint finger0_sensor1_joint
- removed joint finger1_sensor2_joint
- joint finger0_segment0_joint: origin xyz=0.02675 0 0.0 rpy=0 0 0 -> xyz=0.03175 0 0.0 rpy=0 0 0
- joint finger0_segment1_joint: origin xyz=0 0.0936 0 rpy=0 0 0 -> xyz=0 0.072 0 rpy=0 0 0
- joint finger1_segment0_joint: origin xyz=-0.02675 0 3.27593018771917e-18 rpy=0 0 0 -> xyz=-0.03175 0 3.888253587292846e-18 rpy=0 0 0
- joint finger1_segment1_joint: origin xyz=0 0.0936 0 rpy=0 0 0 -> xyz=0 0.072 0 rpy=0 0 0

File: demos/rl_demo/resources/NigelHands/2v2_50.50_50.50_1.1_73/hand/2v2_50.50_50.50_1.1_73.urdf (robot description, URDF)
Before this commit: robot 2v2_65.35_65.35_1.1_53, 7 links, 6 joints
Links:
- removed link finger0_sensor
- removed link finger1_sensor
- link finger0_segment0: mass 0.1 -> None
- link finger0_segment1: mass 0.1 -> None
- link finger1_segment0: mass 0.1 -> None
- link finger1_segment1: mass 0.1 -> None
- link palm: mass 1 -> None
Joints:
- removed joint finger0_sensor1_joint
- removed joint finger1_sensor2_joint
- joint finger0_segment0_joint: origin xyz=0.02675 0 0.0 rpy=0 0 0 -> xyz=0.03675 0 0.0 rpy=0 0 0
- joint finger0_segment1_joint: origin xyz=0 0.0936 0 rpy=0 0 0 -> xyz=0 0.072 0 rpy=0 0 0
- joint finger1_segment0_joint: origin xyz=-0.02675 0 3.27593018771917e-18 rpy=0 0 0 -> xyz=-0.03675 0 4.500576986866523e-18 rpy=0 0 0
- joint finger1_segment1_joint: origin xyz=0 0.0936 0 rpy=0 0 0 -> xyz=0 0.072 0 rpy=0 0 0
