Commit message: updated gui to allow for transfer, fixed hand b dimensions for sensors, updated ddpgfd for runs without rollout

File: demos/rl_demo/resources/2v2_Hand_B/hand/2v2_65.35_65.35_1.1_53.urdf (robot description, URDF)
Before this commit: robot 2v2_65.35_65.35_1.1_53, 7 links, 6 joints
Links:
- link finger0_sensor: geometry collision box size=0 0 0
- link finger1_sensor: geometry collision box size=0 0 0
Joints:
- joint finger0_sensor1_joint: origin xyz=0 0.072 0 rpy=0 0 0 -> xyz=0 0.0504 0 rpy=0 0 0
- joint finger1_sensor2_joint: origin xyz=0 0.072 0 rpy=0 0 0 -> xyz=0 0.0504 0 rpy=0 0 0
