Commit message: updated multiprocessor to work with new RNN gui, wrote some plotting scripts

File: demos/rl_demo/resources/NigelHands/2v2_50.50_50.50_1.1_53/hand/2v2_50.50_50.50_1.1_53.urdf (robot description, URDF)
Before this commit: robot 2v2_50.50_50.50_1.1_53, 5 links, 4 joints
Links:
- added link finger0_sensor, mass 0.000001
- added link finger1_sensor, mass 0.000001
- link finger0_segment0: mass None -> 0.1
- link finger0_segment1: mass None -> 0.1
- link finger1_segment0: mass None -> 0.1
- link finger1_segment1: mass None -> 0.1
- link palm: mass None -> 1
Joints:
- added joint finger0_sensor1_joint: type fixed, parent finger0_segment1, child finger0_sensor, origin xyz=0 0.072 0 rpy=0 0 0, axis 0 0 1, limit lower=-3.14 upper=3.14 effort=1000.0 velocity=0.5
- added joint finger1_sensor2_joint: type fixed, parent finger1_segment1, child finger1_sensor, origin xyz=0 0.072 0 rpy=0 0 0, axis 0 0 1, limit lower=-3.14 upper=3.14 effort=1000.0 velocity=0.5
