Commit message: updated main hands in hand bank to have accurate finger tip poses, fixed a couple bugs in multiprocess run

File: demos/rl_demo/resources/hand_bank/2v2_65.35_65.35_1.1_63/hand/2v2_65.35_65.35_1.1_63.urdf (robot description, URDF)
Before this commit: robot 2v2_65.35_65.35_1.1_63, 7 links, 6 joints
Joints:
- joint finger0_sensor1_joint: origin xyz=0 0.072 0 rpy=0 0 0 -> xyz=0 0.0504 0 rpy=0 0 0
- joint finger1_sensor2_joint: origin xyz=0 0.072 0 rpy=0 0 0 -> xyz=0 0.0504 0 rpy=0 0 0

File: demos/rl_demo/resources/hand_bank/2v2_65.35_65.35_1.1_73/hand/2v2_65.35_65.35_1.1_73.urdf (robot description, URDF)
Before this commit: robot 2v2_65.35_65.35_1.1_73, 7 links, 6 joints
Joints:
- joint finger0_sensor1_joint: origin xyz=0 0.072 0 rpy=0 0 0 -> xyz=0 0.0504 0 rpy=0 0 0
- joint finger1_sensor2_joint: origin xyz=0 0.072 0 rpy=0 0 0 -> xyz=0 0.0504 0 rpy=0 0 0

File: demos/rl_demo/resources/hand_bank/2v2_70.30_70.30_1.1_53/hand/2v2_70.30_70.30_1.1_53.urdf (robot description, URDF)
Before this commit: robot 2v2_70.30_70.30_1.1_53, 7 links, 6 joints
Joints:
- joint finger0_sensor1_joint: origin xyz=0 0.072 0 rpy=0 0 0 -> xyz=0 0.0432 0 rpy=0 0 0
- joint finger1_sensor2_joint: origin xyz=0 0.072 0 rpy=0 0 0 -> xyz=0 0.0432 0 rpy=0 0 0

File: demos/rl_demo/resources/hand_bank/2v2_70.30_70.30_1.1_63/hand/2v2_70.30_70.30_1.1_63.urdf (robot description, URDF)
Before this commit: robot 2v2_70.30_70.30_1.1_63, 7 links, 6 joints
Joints:
- joint finger0_sensor1_joint: origin xyz=0 0.072 0 rpy=0 0 0 -> xyz=0 0.0432 0 rpy=0 0 0
- joint finger1_sensor2_joint: origin xyz=0 0.072 0 rpy=0 0 0 -> xyz=0 0.0432 0 rpy=0 0 0

File: demos/rl_demo/resources/hand_bank/2v2_70.30_70.30_1.1_73/hand/2v2_70.30_70.30_1.1_73.urdf (robot description, URDF)
Before this commit: robot 2v2_70.30_70.30_1.1_73, 7 links, 6 joints
Joints:
- joint finger0_sensor1_joint: origin xyz=0 0.072 0 rpy=0 0 0 -> xyz=0 0.0432 0 rpy=0 0 0
- joint finger1_sensor2_joint: origin xyz=0 0.072 0 rpy=0 0 0 -> xyz=0 0.0432 0 rpy=0 0 0
