Commit message: added domain randomization, cleaned up a lot of stuff

File: demos/rl_demo/resources/hand_bank/2v2_50.50_50.50_1.1_53/hand/2v2_50.50_50.50_1.1_53.urdf (robot description, URDF)
Before this commit: robot 2v2_50.50_50.50_1.1_53, 7 links, 6 joints
Joints:
- joint finger0_segment0_joint: limit lower=-3.14 upper=3.14 effort=1000.0 velocity=0.5 -> lower=-3.14 upper=3.14 effort=1000.0 velocity=0.0005
