Commit message: added to wall task and finalized domain randomization stuff

File: demos/rl_demo/resources/object_models/wallthing/vertical_wall.urdf (robot description, URDF)
Before this commit: robot 2v2_mod_cuboid_large, 1 links, 0 joints
Links:
- link 2v2_mod_cuboid_large: geometry collision mesh filename=obj_files/2v2_mod_cuboid_large_collision.obj scale=1 0.2 0.2; visual mesh filename=obj_files/2v2_mod_cuboid_large_collision.obj scale=1 0.2 0.2
