Commit message: fixed gui and updated URDF to .STL from .stl

File: demos/rl_demo/resources/object_models/Jeremiah_Shapes/20_r_circle.urdf (robot description, URDF)
Before this commit: robot Jeremiah_20_r_circle, 1 links, 0 joints
Links:
- link 20_r_circle: geometry collision mesh filename=Shapes/20_r_circle.STL scale=1 1 1; visual mesh filename=Shapes/20_r_circle.STL scale=1 1 1

File: demos/rl_demo/resources/object_models/Jeremiah_Shapes/20_r_hourglass.urdf (robot description, URDF)
Before this commit: robot Jeremiah_20_r_hourglass, 1 links, 0 joints
Links:
- link 20_r_hourglass: geometry collision mesh filename=Shapes/20_r_hourglass.STL scale=1 1 1; visual mesh filename=Shapes/20_r_hourglass.STL scale=1 1 1

File: demos/rl_demo/resources/object_models/Jeremiah_Shapes/20x12p5_ellipse.urdf (robot description, URDF)
Before this commit: robot Jeremiah_20x12p5_ellipse, 1 links, 0 joints
Links:
- link 20x12p5_ellipse: geometry collision mesh filename=Shapes/20x12p5_ellipse.STL scale=1 1 1; visual mesh filename=Shapes/20x12p5_ellipse.STL scale=1 1 1

File: demos/rl_demo/resources/object_models/Jeremiah_Shapes/40_square_40_concave.urdf (robot description, URDF)
Before this commit: robot Jeremiah_40_square_40_concave, 1 links, 0 joints
Links:
- link 40_square_40_concave: geometry collision mesh filename=Shapes/40_square_40_concave.STL scale=1 1 1; visual mesh filename=Shapes/40_square_40_concave.STL scale=1 1 1

File: demos/rl_demo/resources/object_models/Jeremiah_Shapes/40x40_square.urdf (robot description, URDF)
Before this commit: robot Jeremiah_40x40_Square, 1 links, 0 joints
Links:
- link 40x40_Square: geometry collision mesh filename=Shapes/40x40_Square.STL scale=1 1 1; visual mesh filename=Shapes/40x40_Square.STL scale=1 1 1

File: demos/rl_demo/resources/object_models/Jeremiah_Shapes/40x40_triangle.urdf (robot description, URDF)
Before this commit: robot Jeremiah_40x40_Triangle, 1 links, 0 joints
Links:
- link 40x40_Triangle: geometry collision mesh filename=Shapes/40x40_Triangle.STL scale=1 1 1; visual mesh filename=Shapes/40x40_Triangle.STL scale=1 1 1

File: demos/rl_demo/resources/object_models/Jeremiah_Shapes/45_10_slope_cone.urdf (robot description, URDF)
Before this commit: robot Jeremiah_45_10_slope_cone, 1 links, 0 joints
Links:
- removed link 50x30_Teardrop
- added link 45_10_slope_cone; collision mesh filename=Shapes/45_10_slope_cone.STL scale=1 1 1; visual mesh filename=Shapes/45_10_slope_cone.STL scale=1 1 1

File: demos/rl_demo/resources/object_models/Jeremiah_Shapes/50x30_teardrop.urdf (robot description, URDF)
Before this commit: robot Jeremiah_50x30_Teardrop, 1 links, 0 joints
Links:
- link 50x30_Teardrop: geometry collision mesh filename=Shapes/50x30_Teardrop.STL scale=1 1 1; visual mesh filename=Shapes/50x30_Teardrop.STL scale=1 1 1

Commit message: fixed urdf/stl files for shapes (except 40x40square)

File: demos/rl_demo/resources/object_models/Jeremiah_Shapes/20_r_circle.urdf (robot description, URDF)
Before this commit: robot 20_r_circle, 1 links, 0 joints
Links:
- link 20_r_circle: mass None -> 0.3; geometry collision mesh filename=Shapes/20_r_circle.STL scale=.001 .001 .001; visual mesh filename=Shapes/20_r_circle.STL scale=.001 .001 .001

File: demos/rl_demo/resources/object_models/Jeremiah_Shapes/20_r_hourglass.urdf (robot description, URDF)
Before this commit: robot 20_r_hourglass, 1 links, 0 joints
Links:
- link 20_r_hourglass: mass None -> 0.3; geometry collision mesh filename=Shapes/20_r_hourglass.STL scale=.001 .001 .001; visual mesh filename=Shapes/20_r_hourglass.STL scale=.001 .001 .001

File: demos/rl_demo/resources/object_models/Jeremiah_Shapes/20x12p5_ellipse.urdf (robot description, URDF)
Before this commit: robot 20x12p5_ellipse, 1 links, 0 joints
Links:
- link 20x12p5_ellipse: mass None -> 0.3; geometry collision mesh filename=Shapes/20x12p5_ellipse.STL scale=.001 .001 .001; visual mesh filename=Shapes/20x12p5_ellipse.STL scale=.001 .001 .001

File: demos/rl_demo/resources/object_models/Jeremiah_Shapes/40_square_40_concave.urdf (robot description, URDF)
Before this commit: robot 40_square_40_concave, 1 links, 0 joints
Links:
- link 40_square_40_concave: mass None -> 0.3; geometry collision mesh filename=Shapes/40_square_40_concave.STL scale=.001 .001 .001; visual mesh filename=Shapes/40_square_40_concave.STL scale=.001 .001 .001

File: demos/rl_demo/resources/object_models/Jeremiah_Shapes/40x40_square.urdf (robot description, URDF)
Before this commit: robot 40x40_Square, 1 links, 0 joints
Links:
- link 40x40_Square: mass None -> 0.3; geometry collision mesh filename=Shapes/40x40_square.STL scale=.001 .001 .001; visual mesh filename=Shapes/40x40_square.STL scale=.001 .001 .001

File: demos/rl_demo/resources/object_models/Jeremiah_Shapes/40x40_triangle.urdf (robot description, URDF)
Before this commit: robot 40x40_Triangle, 1 links, 0 joints
Links:
- link 40x40_Triangle: mass None -> 0.3; geometry collision mesh filename=Shapes/40x40_triangle.STL scale=.001 .001 .001; visual mesh filename=Shapes/40x40_triangle.STL scale=.001 .001 .001

File: demos/rl_demo/resources/object_models/Jeremiah_Shapes/45_10_slope_cone.urdf (robot description, URDF)
Before this commit: robot 45_10_slope_cone, 1 links, 0 joints
Links:
- link 45_10_slope_cone: mass None -> 0.3; geometry collision mesh filename=Shapes/45_10_slope_cone.STL scale=.001 .001 .001; visual mesh filename=Shapes/45_10_slope_cone.STL scale=.001 .001 .001

File: demos/rl_demo/resources/object_models/Jeremiah_Shapes/50x30_teardrop.urdf (robot description, URDF)
Before this commit: robot 50x30_Teardrop, 1 links, 0 joints
Links:
- link 50x30_Teardrop: mass None -> 0.3; geometry collision mesh filename=Shapes/50x30_teardrop.STL scale=.001 .001 .001; visual mesh filename=Shapes/50x30_teardrop.STL scale=.001 .001 .001

Commit message: Updated Jeremiahs Shapes and point generator

File: demos/rl_demo/resources/object_models/Jeremiah_Shapes/20_r_circle.urdf (robot description, URDF)
Before this commit: robot 20_r_circle, 1 links, 0 joints
Links:
- link 20_r_circle: geometry collision mesh filename=Shapes/20_r_circle.obj scale=1 1 1; visual mesh filename=Shapes/20_r_circle.obj scale=1 1 1
