Commit message: Added the aspect ratio shapes and bent the RNN gui to my will for implementation. Also added noise to the starting position of the object.

File: demos/rl_demo/resources/object_models/Jeremiah_Shapes/40x40_square_25.urdf (robot description, URDF)
Before this commit: robot 20_r_circle, 1 links, 0 joints
Links:
- removed link 20_r_circle
- added link 40x40_Square, mass 0.3; collision mesh filename=Shapes/40x40_square.obj scale=1.265 1 0.506; visual mesh filename=Shapes/40x40_square.obj scale=1.265 1 0.506
