Commit message: updated URDFs

File: demos/rl_demo/resources/object_models/Jeremiah_Shapes/50x30_teardrop_15.urdf (robot description, URDF)
Before this commit: robot 50x30_Teardrop, 1 links, 0 joints
Links:
- link 50x30_Teardrop: geometry collision mesh filename=Shapes/50x30_teardrop.obj scale=0.5443 1 0.8165; visual mesh filename=Shapes/50x30_teardrop.obj scale=0.5443 1 0.8165

File: demos/rl_demo/resources/object_models/Jeremiah_Shapes/50x30_teardrop_2.urdf (robot description, URDF)
Before this commit: robot 50x30_Teardrop, 1 links, 0 joints
Links:
- link 50x30_Teardrop: geometry collision mesh filename=Shapes/50x30_teardrop.obj scale=0.3535 1 0.707; visual mesh filename=Shapes/50x30_teardrop.obj scale=0.3535 1 0.707

File: demos/rl_demo/resources/object_models/Jeremiah_Shapes/50x30_teardrop_25.urdf (robot description, URDF)
Before this commit: robot 50x30_Teardrop, 1 links, 0 joints
Links:
- link 50x30_Teardrop: geometry collision mesh filename=Shapes/50x30_teardrop.obj scale=0.506 1 1.265; visual mesh filename=Shapes/50x30_teardrop.obj scale=0.506 1 1.265

File: demos/rl_demo/resources/object_models/Jeremiah_Shapes/50x30_teardrop_3.urdf (robot description, URDF)
Before this commit: robot 50x30_Teardrop, 1 links, 0 joints
Links:
- link 50x30_Teardrop: geometry collision mesh filename=Shapes/50x30_teardrop.obj scale=0.385 1 1.1546; visual mesh filename=Shapes/50x30_teardrop.obj scale=0.385 1 1.1546

Commit message: Updated Teardrop to be more consistent, created training data generator and slices.json

File: demos/rl_demo/resources/object_models/Jeremiah_Shapes/50x30_teardrop_15.urdf (robot description, URDF)
Before this commit: robot 50x30_Teardrop, 1 links, 0 joints
Links:
- link 50x30_Teardrop: geometry collision mesh filename=Shapes/50x30_teardrop.obj scale=0.8165 1 0.5443; visual mesh filename=Shapes/50x30_teardrop.obj scale=0.8165 1 0.5443

File: demos/rl_demo/resources/object_models/Jeremiah_Shapes/50x30_teardrop_2.urdf (robot description, URDF)
Before this commit: robot 50x30_Teardrop, 1 links, 0 joints
Links:
- link 50x30_Teardrop: geometry collision mesh filename=Shapes/50x30_teardrop.obj scale=0.707 1 0.3535; visual mesh filename=Shapes/50x30_teardrop.obj scale=0.707 1 0.3535

File: demos/rl_demo/resources/object_models/Jeremiah_Shapes/50x30_teardrop_25.urdf (robot description, URDF)
Before this commit: robot 50x30_Teardrop, 1 links, 0 joints
Links:
- link 50x30_Teardrop: geometry collision mesh filename=Shapes/50x30_teardrop.obj scale=1.265 1 0.506; visual mesh filename=Shapes/50x30_teardrop.obj scale=1.265 1 0.506

File: demos/rl_demo/resources/object_models/Jeremiah_Shapes/50x30_teardrop_3.urdf (robot description, URDF)
Before this commit: robot 50x30_Teardrop, 1 links, 0 joints
Links:
- link 50x30_Teardrop: geometry collision mesh filename=Shapes/50x30_teardrop.obj scale=1.1546 1 0.385; visual mesh filename=Shapes/50x30_teardrop.obj scale=1.1546 1 0.385
