Commit message: Updated the RNNGui with new shapes. Added new shapes.

File: demos/rl_demo/resources/object_models/Jeremiah_Shapes/pentagon_15.urdf (robot description, URDF)
Before this commit: robot pentagon, 1 links, 0 joints
Links:
- link pentagon: geometry collision mesh filename=Shapes/pentagon.obj scale=0.05443 .1 0.08165; visual mesh filename=Shapes/pentagon.obj scale=0.05443 .1 0.08165

File: demos/rl_demo/resources/object_models/Jeremiah_Shapes/pentagon_2.urdf (robot description, URDF)
Before this commit: robot pentagon, 1 links, 0 joints
Links:
- link pentagon: geometry collision mesh filename=Shapes/pentagon.obj scale=0.03535 .1 0.0707; visual mesh filename=Shapes/pentagon.obj scale=0.03535 .1 0.0707

File: demos/rl_demo/resources/object_models/Jeremiah_Shapes/pentagon_3.urdf (robot description, URDF)
Before this commit: robot pentagon, 1 links, 0 joints
Links:
- link pentagon: geometry collision mesh filename=Shapes/pentagon.obj scale=0.0385 .1 0.11546; visual mesh filename=Shapes/pentagon.obj scale=0.0385 .1 0.11546
